File: I2C-ToF-Companion.kicad_pcb (KiCad board)
At the start: 2 copper layers, 24.4 x 12.7 mm, 10 parts, among them IC1 LTC4316CMS#PBF, J1 Conn_01x04, J2 Conn_01x04

Commit message: Final v1.0 version
Parts:
- J1, J2: footprint Connector_JST:JST_SH_SM04B-SRSS-TB_1x04-1MP_P1.00mm_Horizontal -> Connector_JST:JST_SH_BM04B-SRSS-TB_1x04-1MP_P1.00mm_Vertical
- moved J1 0.40 mm to (157.3, 75.4), turned to -90 degrees
- moved J2 0.35 mm to (139.8, 75.4), turned to 90 degrees
Routing:
- net /GND: track 4.00 -> 9.52 mm
- net /SDA: track 28.2 -> 32.9 mm
- net /SCL: track 33.3 -> 36.9 mm
- net /3.3v: track 46.3 -> 47.8 mm
Other:
- board size 24.4 x 12.7 mm -> 22 x 12.7 mm
